File: valve_reporter.sch (KiCad schematic (older format))
At the start: 52 parts, among them J1 Screw_Terminal_01x05, J2 Screw_Terminal_01x14, K1 G5LE-1, Q1 2N3904, U1 NodeMCU_1.0_(ESP-12E), U2 MC7805CTG

Commit message: Created layout
Parts:
- D10, D11, D12, D13, D14, D15, D16: footprint digikey-footprints:DO-214AC -> Diode_SMD:D_SOD-323_HandSoldering
Changed lines of the file:
@@
 F 0 "D16" V 7854 4379 50  0000 L CNN
 F 1 "D_Shockley" V 7945 4379 50  0000 L CNN
-F 2 "digikey-footprints:DO-214AC" H 7900 4300 50  0001 C CNN
+F 2 "Diode_SMD:D_SOD-323_HandSoldering" H 7900 4300 50  0001 C CNN
 F 3 "~" H 7900 4300 50  0001 C CNN
 	1    7900 4300
@@
 F 0 "D15" V 7804 3829 50  0000 L CNN
 F 1 "D_Shockley" V 7895 3829 50  0000 L CNN
-F 2 "digikey-footprints:DO-214AC" H 7850 3750 50  0001 C CNN
+F 2 "Diode_SMD:D_SOD-323_HandSoldering" H 7850 3750 50  0001 C CNN
 F 3 "~" H 7850 3750 50  0001 C CNN
 	1    7850 3750
@@
 F 0 "D14" V 7804 3279 50  0000 L CNN
 F 1 "D_Shockley" V 7895 3279 50  0000 L CNN
-F 2 "digikey-footprints:DO-214AC" H 7850 3200 50  0001 C CNN
+F 2 "Diode_SMD:D_SOD-323_HandSoldering" H 7850 3200 50  0001 C CNN
 F 3 "~" H 7850 3200 50  0001 C CNN
 	1    7850 3200
@@
 F 0 "D13" V 7804 2729 50  0000 L CNN
 F 1 "D_Shockley" V 7895 2729 50  0000 L CNN
-F 2 "digikey-footprints:DO-214AC" H 7850 2650 50  0001 C CNN
+F 2 "Diode_SMD:D_SOD-323_HandSoldering" H 7850 2650 50  0001 C CNN
 F 3 "~" H 7850 2650 50  0001 C CNN
 	1    7850 2650
@@
 F 0 "D12" V 7804 2179 50  0000 L CNN
 F 1 "D_Shockley" V 7895 2179 50  0000 L CNN
-F 2 "digikey-footprints:DO-214AC" H 7850 2100 50  0001 C CNN
+F 2 "Diode_SMD:D_SOD-323_HandSoldering" H 7850 2100 50  0001 C CNN
 F 3 "~" H 7850 2100 50  0001 C CNN
 	1    7850 2100
@@
 F 0 "D11" V 7804 1629 50  0000 L CNN
 F 1 "D_Shockley" V 7895 1629 50  0000 L CNN
-F 2 "digikey-footprints:DO-214AC" H 7850 1550 50  0001 C CNN
+F 2 "Diode_SMD:D_SOD-323_HandSoldering" H 7850 1550 50  0001 C CNN
 F 3 "~" H 7850 1550 50  0001 C CNN
 	1    7850 1550
@@
 F 0 "D10" V 7804 1079 50  0000 L CNN
 F 1 "D_Shockley" V 7895 1079 50  0000 L CNN
-F 2 "digikey-footprints:DO-214AC" H 7850 1000 50  0001 C CNN
+F 2 "Diode_SMD:D_SOD-323_HandSoldering" H 7850 1000 50  0001 C CNN
 F 3 "~" H 7850 1000 50  0001 C CNN
 	1    7850 1000

Commit message: Schematic is shaping up
Parts:
- added H5, H6, H7, H8: MountingHole_Pad, MountingHole:MountingHole_3.2mm_M3_ISO7380_Pad, symbol Mechanical:MountingHole_Pad
- D3, D4, D5, D6, D7, D8, D9: footprint Diode_SMD:D_SOD-323F -> Diode_SMD:D_SOD-323_HandSoldering
- J1: footprint TerminalBlock_Phoenix:TerminalBlock_Phoenix_PT-1,5-5-5.0-H_1x05_P5.00mm_Horizontal -> TerminalBlock_Phoenix:TerminalBlock_Phoenix_PT-1,5-5-5.0-H_1x05_P5.00mm_Horizontal_valve_rep
- J2: footprint TerminalBlock_Phoenix:TerminalBlock_Phoenix_PT-1,5-14-3.5-H_1x14_P3.50mm_Horizontal -> TerminalBlock_Phoenix:TerminalBlock_Phoenix_PT-1,5-14-3.5-H_1x14_P3.50mm_Horizontal_valve_rep
Connections:
- net +12V: now also J2.10 (Pin_10), J2.12 (Pin_12), J2.14 (Pin_14), J2.2 (Pin_2), J2.4 (Pin_4), J2.6 (Pin_6), J2.8 (Pin_8); no longer J2.1 (Pin_1), J2.11 (Pin_11), J2.13 (Pin_13), J2.3 (Pin_3), J2.5 (Pin_5), J2.7 (Pin_7), J2.9 (Pin_9)
- net GND: now also H5.1, H6.1, H7.1, H8.1
- net at D14.1 (K), R14.1: now also J2.5 (Pin_5); no longer J2.10 (Pin_10)
- net at D15.1 (K), R15.1: now also J2.3 (Pin_3); no longer J2.12 (Pin_12)
- net at D16.1 (K), R16.1: now also J2.1 (Pin_1); no longer J2.14 (Pin_14)
- net at D10.1 (K), R10.1: now also J2.13 (Pin_13); no longer J2.2 (Pin_2)
- net at D11.1 (K), R11.1: now also J2.11 (Pin_11); no longer J2.4 (Pin_4)
- net at D12.1 (K), R12.1: now also J2.9 (Pin_9); no longer J2.6 (Pin_6)
- net at D13.1 (K), R13.1: now also J2.7 (Pin_7); no longer J2.8 (Pin_8)
- net RelIn: now reaches J1.5 (Pin_5), K1.1
- net RelOff: now reaches J1.4 (Pin_4), K1.3
- net RelOn: now reaches J1.3 (Pin_3), K1.4
Other:
- moved on the sheet: J2
Changed lines of the file:
@@
 L Connector:Screw_Terminal_01x14 J2
 U 1 1 5C4F2851
-P 10250 3800
-F 0 "J2" H 10330 3792 50  0000 L CNN
-F 1 "Screw_Terminal_01x14" H 10330 3701 50  0000 L CNN
-F 2 "TerminalBlock_Phoenix:TerminalBlock_Phoenix_PT-1,5-14-3.5-H_1x14_P3.50mm_Horizontal" H 10250 3800 50  0001 C CNN
-F 3 "~" H 10250 3800 50  0001 C CNN
-	1    10250 3800
-	1    0    0    -1
+P 10150 3900
+F 0 "J2" H 10230 3892 50  0000 L CNN
+F 1 "Screw_Terminal_01x14" H 10230 3801 50  0000 L CNN
+F 2 "TerminalBlock_Phoenix:TerminalBlock_Phoenix_PT-1,5-14-3.5-H_1x14_P3.50mm_Horizontal_valve_rep" H 10150 3900 50  0001 C CNN
+F 3 "~" H 10150 3900 50  0001 C CNN
+	1    10150 3900
+	1    0    0    1
 $EndComp
 $Comp
 L power:+12V #PWR0110
 U 1 1 5C4F28B4
-P 9900 3050
-F 0 "#PWR0110" H 9900 2900 50  0001 C CNN
-F 1 "+12V" H 9915 3223 50  0000 C CNN
-F 2 "" H 9900 3050 50  0001 C CNN
-F 3 "" H 9900 3050 50  0001 C CNN
-	1    9900 3050
-	1    0    0    -1
-$EndComp
-Wire Wire Line
-	10050 3200 9900 3200
-Wire Wire Line
-	9900 3200 9900 3050
-Wire Wire Line
-	10050 3400 9900 3400
-Wire Wire Line
-	9900 3400 9900 3200
-Connection ~ 9900 3200
-Wire Wire Line
-	10050 3600 9900 3600
-Wire Wire Line
-	9900 3600 9900 3400
-Connection ~ 9900 3400
-Wire Wire Line
-	10050 3800 9900 3800
-Wire Wire Line
-	9900 3800 9900 3600
-Connection ~ 9900 3600
-Wire Wire Line
-	10050 4000 9900 4000
-Wire Wire Line
-	9900 4000 9900 3800
-Connection ~ 9900 3800
-Wire Wire Line
-	10050 4200 9900 4200
-Wire Wire Line
-	9900 4200 9900 4000
-Connection ~ 9900 4000
-Wire Wire Line
-	10050 4400 9900 4400
-Wire Wire Line
-	9900 4400 9900 4200
-Connection ~ 9900 4200
+P 9800 3150
+F 0 "#PWR0110" H 9800 3000 50  0001 C CNN
+F 1 "+12V" H 9815 3323 50  0000 C CNN
+F 2 "" H 9800 3150 50  0001 C CNN
+F 3 "" H 9800 3150 50  0001 C CNN
+	1    9800 3150
+	1    0    0    -1
+$EndComp
 $Comp
 L Device:R R16
@@
 F 0 "D9" V 7404 4379 50  0000 L CNN
 F 1 "3.3V" V 7495 4379 50  0000 L CNN
-F 2 "Diode_SMD:D_SOD-323F" H 7450 4300 50  0001 C CNN
+F 2 "Diode_SMD:D_SOD-323_HandSoldering" H 7450 4300 50  0001 C CNN
 F 3 "~" H 7450 4300 50  0001 C CNN
 	1    7450 4300
@@
 F 0 "D8" V 7354 3829 50  0000 L CNN
 F 1 "3.3V" V 7445 3829 50  0000 L CNN
-F 2 "Diode_SMD:D_SOD-323F" H 7400 3750 50  0001 C CNN
+F 2 "Diode_SMD:D_SOD-323_HandSoldering" H 7400 3750 50  0001 C CNN
 F 3 "~" H 7400 3750 50  0001 C CNN
 	1    7400 3750
@@
 F 0 "D7" V 7354 3279 50  0000 L CNN
 F 1 "3.3V" V 7445 3279 50  0000 L CNN
-F 2 "Diode_SMD:D_SOD-323F" H 7400 3200 50  0001 C CNN
+F 2 "Diode_SMD:D_SOD-323_HandSoldering" H 7400 3200 50  0001 C CNN
 F 3 "~" H 7400 3200 50  0001 C CNN
 	1    7400 3200
@@
 F 0 "D6" V 7354 2729 50  0000 L CNN
 F 1 "3.3V" V 7445 2729 50  0000 L CNN
-F 2 "Diode_SMD:D_SOD-323F" H 7400 2650 50  0001 C CNN
+F 2 "Diode_SMD:D_SOD-323_HandSoldering" H 7400 2650 50  0001 C CNN
 F 3 "~" H 7400 2650 50  0001 C CNN
 	1    7400 2650
@@
 F 0 "D5" V 7354 2179 50  0000 L CNN
 F 1 "3.3V" V 7445 2179 50  0000 L CNN
-F 2 "Diode_SMD:D_SOD-323F" H 7400 2100 50  0001 C CNN
+F 2 "Diode_SMD:D_SOD-323_HandSoldering" H 7400 2100 50  0001 C CNN
 F 3 "~" H 7400 2100 50  0001 C CNN
 	1    7400 2100
@@
 F 0 "D4" V 7354 1629 50  0000 L CNN
 F 1 "3.3V" V 7445 1629 50  0000 L CNN
-F 2 "Diode_SMD:D_SOD-323F" H 7400 1550 50  0001 C CNN
+F 2 "Diode_SMD:D_SOD-323_HandSoldering" H 7400 1550 50  0001 C CNN
 F 3 "~" H 7400 1550 50  0001 C CNN
 	1    7400 1550
@@
 F 0 "D3" V 7354 1079 50  0000 L CNN
 F 1 "3.3V" V 7445 1079 50  0000 L CNN
-F 2 "Diode_SMD:D_SOD-323F" H 7400 1000 50  0001 C CNN
+F 2 "Diode_SMD:D_SOD-323_HandSoldering" H 7400 1000 50  0001 C CNN
 F 3 "~" H 7400 1000 50  0001 C CNN
 	1    7400 1000
@@
 Connection ~ 6800 4150
 Wire Wire Line
-	10050 3300 9700 3300
-Wire Wire Line
 	9700 3300 9700 850
 Wire Wire Line
@@
 Connection ~ 7850 850
 Wire Wire Line
-	10050 3500 9550 3500
-Wire Wire Line
 	9550 3500 9550 1400
 Wire Wire Line
@@
 Connection ~ 7850 1400
 Wire Wire Line
-	10050 3700 9400 3700
-Wire Wire Line
 	9400 3700 9400 1950
 Wire Wire Line
@@
 Connection ~ 7850 1950
 Wire Wire Line
-	10050 3900 9250 3900
-Wire Wire Line
 	9250 3900 9250 2500
 Wire Wire Line
@@
 Connection ~ 7850 2500
 Wire Wire Line
-	10050 4100 9100 4100
-Wire Wire Line
 	9100 4100 9100 3050
 Wire Wire Line
@@
 Connection ~ 7850 3050
 Wire Wire Line
-	10050 4300 8950 4300
-Wire Wire Line
 	8950 4300 8950 3600
 Wire Wire Line
 	8950 3600 7850 3600
 Connection ~ 7850 3600
-Wire Wire Line
-	10050 4500 8800 4500
 Wire Wire Line
 	8800 4500 8800 4150
@@
 L power:GND #PWR0105
 U 1 1 5C7EC909
-P 900 3250
-F 0 "#PWR0105" H 900 3000 50  0001 C CNN
-F 1 "GND" H 905 3077 50  0000 C CNN
-F 2 "" H 900 3250 50  0001 C CNN
-F 3 "" H 900 3250 50  0001 C CNN
-	1    900  3250
-	1    0    0    -1
-$EndComp
-Wire Wire Line
-	900  3250 900  3150
+P 900 4400
+F 0 "#PWR0105" H 900 4150 50  0001 C CNN
+F 1 "GND" H 905 4227 50  0000 C CNN
+F 2 "" H 900 4400 50  0001 C CNN
+F 3 "" H 900 4400 50  0001 C CNN
+	1    900  4400
+	1    0    0    -1
+$EndComp
+Wire Wire Line
+	900  4400 900  4150
 Connection ~ 900  3150
 $Comp
@@
 F 0 "J1" H 7530 5992 50  0000 L CNN
 F 1 "Screw_Terminal_01x05" H 7530 5901 50  0000 L CNN
-F 2 "TerminalBlock_Phoenix:TerminalBlock_Phoenix_PT-1,5-5-5.0-H_1x05_P5.00mm_Horizontal" H 7450 5950 50  0001 C CNN
+F 2 "TerminalBlock_Phoenix:TerminalBlock_Phoenix_PT-1,5-5-5.0-H_1x05_P5.00mm_Horizontal_valve_rep" H 7450 5950 50  0001 C CNN
 F 3 "~" H 7450 5950 50  0001 C CNN
 	1    7450 5950
@@
 Wire Wire Line
 	3750 5800 3400 5800
+Wire Wire Line
+	9950 3200 9800 3200
+Wire Wire Line
+	9800 3200 9800 3150
+Wire Wire Line
+	9950 3400 9800 3400
+Wire Wire Line
+	9800 3400 9800 3200
+Connection ~ 9800 3200
+Wire Wire Line
+	9950 3600 9800 3600
+Wire Wire Line
+	9800 3600 9800 3400
+Connection ~ 9800 3400
+Wire Wire Line
+	9950 3800 9800 3800
+Wire Wire Line
+	9800 3800 9800 3600
+Connection ~ 9800 3600
+Wire Wire Line
+	9950 4000 9800 4000
+Wire Wire Line
+	9800 4000 9800 3800
+Connection ~ 9800 3800
+Wire Wire Line
+	9950 4200 9800 4200
+Wire Wire Line
+	9800 4200 9800 4000
+Connection ~ 9800 4000
+Wire Wire Line
+	9950 4400 9800 4400
+Wire Wire Line
+	9800 4400 9800 4200
+Connection ~ 9800 4200
+Wire Wire Line
+	9950 3300 9700 3300
+Wire Wire Line
+	9950 3500 9550 3500
+Wire Wire Line
+	9950 3700 9400 3700
+Wire Wire Line
+	9950 3900 9250 3900
+Wire Wire Line
+	9950 4100 9100 4100
+Wire Wire Line
+	9950 4300 8950 4300
+Wire Wire Line
+	9950 4500 8800 4500
+$Comp
+L Mechanical:MountingHole_Pad H5
+U 1 1 5C605589
+P 1000 3400
+F 0 "H5" V 954 3550 50  0000 L CNN
+F 1 "MountingHole_Pad" V 1045 3550 50  0000 L CNN
+F 2 "MountingHole:MountingHole_3.2mm_M3_ISO7380_Pad" H 1000 3400 50  0001 C CNN
+F 3 "~" H 1000 3400 50  0001 C CNN
+	1    1000 3400
+	0    1    1    0
+$EndComp
+$Comp
+L Mechanical:MountingHole_Pad H6
+U 1 1 5C605611
+P 1000 3650
+F 0 "H6" V 954 3800 50  0000 L CNN
+F 1 "MountingHole_Pad" V 1045 3800 50  0000 L CNN
+F 2 "MountingHole:MountingHole_3.2mm_M3_ISO7380_Pad" H 1000 3650 50  0001 C CNN
+F 3 "~" H 1000 3650 50  0001 C CNN
+	1    1000 3650
+	0    1    1    0
+$EndComp
+$Comp
+L Mechanical:MountingHole_Pad H7
+U 1 1 5C605747
+P 1000 3900
+F 0 "H7" V 954 4050 50  0000 L CNN
+F 1 "MountingHole_Pad" V 1045 4050 50  0000 L CNN
+F 2 "MountingHole:MountingHole_3.2mm_M3_ISO7380_Pad" H 1000 3900 50  0001 C CNN
+F 3 "~" H 1000 3900 50  0001 C CNN
+	1    1000 3900
+	0    1    1    0
+$EndComp
+$Comp
+L Mechanical:MountingHole_Pad H8
+U 1 1 5C6057D5
+P 1000 4150
+F 0 "H8" V 954 4300 50  0000 L CNN
+F 1 "MountingHole_Pad" V 1045 4300 50  0000 L CNN
+F 2 "MountingHole:MountingHole_3.2mm_M3_ISO7380_Pad" H 1000 4150 50  0001 C CNN
+F 3 "~" H 1000 4150 50  0001 C CNN
+	1    1000 4150
+	0    1    1    0
+$EndComp
+Connection ~ 900  3400
+Wire Wire Line
+	900  3400 900  3150
+Connection ~ 900  3650
+Wire Wire Line
+	900  3650 900  3400
+Connection ~ 900  3900
+Wire Wire Line
+	900  3900 900  3650
+Connection ~ 900  4150
+Wire Wire Line
+	900  4150 900  3900
+Text Label 6850 5800 0    50   ~ 0
+RelOn
+Text Label 6900 6050 0    50   ~ 0
+RelOff
+Text Label 6550 6250 0    50   ~ 0
+RelIn
+Text Label 5400 5600 0    50   ~ 0
+RelDrive
 $EndSCHEMATC

Commit message: Extra decoupling
Parts:
- added C10: 50uF, Capacitor_SMD:C_2816_7142Metric_Pad3.20x4.45mm_HandSolder, symbol Device:C_Small
Connections:
- net +12V: now also C10.1
- net GND: now also C10.2
Changed lines of the file:
@@
 Text Label 5400 5600 0    50   ~ 0
 RelDrive
+$Comp
+L Device:C_Small C10
+U 1 1 5C53AE0A
+P 2400 5100
+F 0 "C10" H 2492 5146 50  0000 L CNN
+F 1 "50uF" H 2492 5055 50  0000 L CNN
+F 2 "Capacitor_SMD:C_2816_7142Metric_Pad3.20x4.45mm_HandSolder" H 2400 5100 50  0001 C CNN
+F 3 "~" H 2400 5100 50  0001 C CNN
+	1    2400 5100
+	1    0    0    -1
+$EndComp
+Wire Wire Line
+	2400 5000 2400 4900
+Wire Wire Line
+	2400 4900 2850 4900
+Connection ~ 2850 4900
+Wire Wire Line
+	2400 5200 2400 5800
+Wire Wire Line
+	2400 5800 2850 5800
+Connection ~ 2850 5800
 $EndSCHEMATC

Commit message: Move to handsolder pads to make live easier
Parts:
- C2, C3, C4, C5, C6, C7, C8, C9: footprint Capacitor_SMD:C_1206_3216Metric -> Capacitor_SMD:C_1206_3216Metric_Pad1.42x1.75mm_HandSolder
- D1: footprint LED_SMD:LED_1206_3216Metric -> LED_SMD:LED_1206_3216Metric_Pad1.42x1.75mm_HandSolder
- D2: footprint Diode_SMD:D_1206_3216Metric -> Diode_SMD:D_1206_3216Metric_Pad1.42x1.75mm_HandSolder
- R1, R10, R11, R12, R13, R14, R15, R16, R17, R2, R3, R4, R5, R6, R7, R8, R9: footprint Resistor_SMD:R_1206_3216Metric -> Resistor_SMD:R_1206_3216Metric_Pad1.42x1.75mm_HandSolder
Changed lines of the file:
@@
 F 0 "R16" V 7493 4150 50  0000 C CNN
 F 1 "1k" V 7584 4150 50  0000 C CNN
-F 2 "Resistor_SMD:R_1206_3216Metric" V 7630 4150 50  0001 C CNN
+F 2 "Resistor_SMD:R_1206_3216Metric_Pad1.42x1.75mm_HandSolder" V 7630 4150 50  0001 C CNN
 F 3 "~" H 7700 4150 50  0001 C CNN
 	1    7700 4150
@@
 F 0 "C7" H 7142 4296 50  0000 L CNN
 F 1 "0.01uF" H 7142 4205 50  0000 L CNN
-F 2 "Capacitor_SMD:C_1206_3216Metric" H 7050 4250 50  0001 C CNN
+F 2 "Capacitor_SMD:C_1206_3216Metric_Pad1.42x1.75mm_HandSolder" H 7050 4250 50  0001 C CNN
 F 3 "~" H 7050 4250 50  0001 C CNN
 	1    7050 4250
@@
 F 0 "R9" H 6730 4254 50  0000 R CNN
 F 1 "1k" H 6730 4345 50  0000 R CNN
-F 2 "Resistor_SMD:R_1206_3216Metric" V 6730 4300 50  0001 C CNN
+F 2 "Resistor_SMD:R_1206_3216Metric_Pad1.42x1.75mm_HandSolder" V 6730 4300 50  0001 C CNN
 F 3 "~" H 6800 4300 50  0001 C CNN
 	1    6800 4300
@@
 F 0 "D2" V 5354 6029 50  0000 L CNN
 F 1 "D" V 5445 6029 50  0000 L CNN
-F 2 "Diode_SMD:D_1206_3216Metric" H 5400 5950 50  0001 C CNN
+F 2 "Diode_SMD:D_1206_3216Metric_Pad1.42x1.75mm_HandSolder" H 5400 5950 50  0001 C CNN
 F 3 "~" H 5400 5950 50  0001 C CNN
 	1    5400 5950
@@
 F 0 "R2" V 4993 6600 50  0000 C CNN
 F 1 "2k" V 5084 6600 50  0000 C CNN
-F 2 "Resistor_SMD:R_1206_3216Metric" V 5130 6600 50  0001 C CNN
+F 2 "Resistor_SMD:R_1206_3216Metric_Pad1.42x1.75mm_HandSolder" V 5130 6600 50  0001 C CNN
 F 3 "~" H 5200 6600 50  0001 C CNN
 	1    5200 6600
@@
 F 0 "R15" V 7443 3600 50  0000 C CNN
 F 1 "1k" V 7534 3600 50  0000 C CNN
-F 2 "Resistor_SMD:R_1206_3216Metric" V 7580 3600 50  0001 C CNN
+F 2 "Resistor_SMD:R_1206_3216Metric_Pad1.42x1.75mm_HandSolder" V 7580 3600 50  0001 C CNN
 F 3 "~" H 7650 3600 50  0001 C CNN
 	1    7650 3600
@@
 F 0 "C6" H 7092 3746 50  0000 L CNN
 F 1 "0.01uF" H 7092 3655 50  0000 L CNN
-F 2 "Capacitor_SMD:C_1206_3216Metric" H 7000 3700 50  0001 C CNN
+F 2 "Capacitor_SMD:C_1206_3216Metric_Pad1.42x1.75mm_HandSolder" H 7000 3700 50  0001 C CNN
 F 3 "~" H 7000 3700 50  0001 C CNN
 	1    7000 3700
@@
 F 0 "R8" H 6680 3704 50  0000 R CNN
 F 1 "1k" H 6680 3795 50  0000 R CNN
-F 2 "Resistor_SMD:R_1206_3216Metric" V 6680 3750 50  0001 C CNN
+F 2 "Resistor_SMD:R_1206_3216Metric_Pad1.42x1.75mm_HandSolder" V 6680 3750 50  0001 C CNN
 F 3 "~" H 6750 3750 50  0001 C CNN
 	1    6750 3750
@@
 F 0 "R14" V 7443 3050 50  0000 C CNN
 F 1 "1k" V 7534 3050 50  0000 C CNN
-F 2 "Resistor_SMD:R_1206_3216Metric" V 7580 3050 50  0001 C CNN
+F 2 "Resistor_SMD:R_1206_3216Metric_Pad1.42x1.75mm_HandSolder" V 7580 3050 50  0001 C CNN
 F 3 "~" H 7650 3050 50  0001 C CNN
 	1    7650 3050
@@
 F 0 "C5" H 7092 3196 50  0000 L CNN
 F 1 "0.01uF" H 7092 3105 50  0000 L CNN
-F 2 "Capacitor_SMD:C_1206_3216Metric" H 7000 3150 50  0001 C CNN
+F 2 "Capacitor_SMD:C_1206_3216Metric_Pad1.42x1.75mm_HandSolder" H 7000 3150 50  0001 C CNN
 F 3 "~" H 7000 3150 50  0001 C CNN
 	1    7000 3150
@@
 F 0 "R7" H 6680 3154 50  0000 R CNN
 F 1 "1k" H 6680 3245 50  0000 R CNN
-F 2 "Resistor_SMD:R_1206_3216Metric" V 6680 3200 50  0001 C CNN
+F 2 "Resistor_SMD:R_1206_3216Metric_Pad1.42x1.75mm_HandSolder" V 6680 3200 50  0001 C CNN
 F 3 "~" H 6750 3200 50  0001 C CNN
 	1    6750 3200
@@
 F 0 "R13" V 7443 2500 50  0000 C CNN
 F 1 "1k" V 7534 2500 50  0000 C CNN
-F 2 "Resistor_SMD:R_1206_3216Metric" V 7580 2500 50  0001 C CNN
+F 2 "Resistor_SMD:R_1206_3216Metric_Pad1.42x1.75mm_HandSolder" V 7580 2500 50  0001 C CNN
 F 3 "~" H 7650 2500 50  0001 C CNN
 	1    7650 2500
@@
 F 0 "C4" H 7092 2646 50  0000 L CNN
 F 1 "0.01uF" H 7092 2555 50  0000 L CNN
-F 2 "Capacitor_SMD:C_1206_3216Metric" H 7000 2600 50  0001 C CNN
+F 2 "Capacitor_SMD:C_1206_3216Metric_Pad1.42x1.75mm_HandSolder" H 7000 2600 50  0001 C CNN
 F 3 "~" H 7000 2600 50  0001 C CNN
 	1    7000 2600
@@
 F 0 "R6" H 6680 2604 50  0000 R CNN
 F 1 "1k" H 6680 2695 50  0000 R CNN
-F 2 "Resistor_SMD:R_1206_3216Metric" V 6680 2650 50  0001 C CNN
+F 2 "Resistor_SMD:R_1206_3216Metric_Pad1.42x1.75mm_HandSolder" V 6680 2650 50  0001 C CNN
 F 3 "~" H 6750 2650 50  0001 C CNN
 	1    6750 2650
@@
 F 0 "R12" V 7443 1950 50  0000 C CNN
 F 1 "1k" V 7534 1950 50  0000 C CNN
-F 2 "Resistor_SMD:R_1206_3216Metric" V 7580 1950 50  0001 C CNN
+F 2 "Resistor_SMD:R_1206_3216Metric_Pad1.42x1.75mm_HandSolder" V 7580 1950 50  0001 C CNN
 F 3 "~" H 7650 1950 50  0001 C CNN
 	1    7650 1950
@@
 F 0 "C3" H 7092 2096 50  0000 L CNN
 F 1 "0.01uF" H 7092 2005 50  0000 L CNN
-F 2 "Capacitor_SMD:C_1206_3216Metric" H 7000 2050 50  0001 C CNN
+F 2 "Capacitor_SMD:C_1206_3216Metric_Pad1.42x1.75mm_HandSolder" H 7000 2050 50  0001 C CNN
 F 3 "~" H 7000 2050 50  0001 C CNN
 	1    7000 2050
@@
 F 0 "R5" H 6680 2054 50  0000 R CNN
 F 1 "1k" H 6680 2145 50  0000 R CNN
-F 2 "Resistor_SMD:R_1206_3216Metric" V 6680 2100 50  0001 C CNN
+F 2 "Resistor_SMD:R_1206_3216Metric_Pad1.42x1.75mm_HandSolder" V 6680 2100 50  0001 C CNN
 F 3 "~" H 6750 2100 50  0001 C CNN
 	1    6750 2100
@@
 F 0 "R11" V 7443 1400 50  0000 C CNN
 F 1 "1k" V 7534 1400 50  0000 C CNN
-F 2 "Resistor_SMD:R_1206_3216Metric" V 7580 1400 50  0001 C CNN
+F 2 "Resistor_SMD:R_1206_3216Metric_Pad1.42x1.75mm_HandSolder" V 7580 1400 50  0001 C CNN
 F 3 "~" H 7650 1400 50  0001 C CNN
 	1    7650 1400
@@
 F 0 "C2" H 7092 1546 50  0000 L CNN
 F 1 "0.01uF" H 7092 1455 50  0000 L CNN
-F 2 "Capacitor_SMD:C_1206_3216Metric" H 7000 1500 50  0001 C CNN
+F 2 "Capacitor_SMD:C_1206_3216Metric_Pad1.42x1.75mm_HandSolder" H 7000 1500 50  0001 C CNN
 F 3 "~" H 7000 1500 50  0001 C CNN
 	1    7000 1500
@@
 F 0 "R4" H 6680 1504 50  0000 R CNN
 F 1 "1k" H 6680 1595 50  0000 R CNN
-F 2 "Resistor_SMD:R_1206_3216Metric" V 6680 1550 50  0001 C CNN
+F 2 "Resistor_SMD:R_1206_3216Metric_Pad1.42x1.75mm_HandSolder" V 6680 1550 50  0001 C CNN
 F 3 "~" H 6750 1550 50  0001 C CNN
 	1    6750 1550
@@
 F 0 "R10" V 7443 850 50  0000 C CNN
 F 1 "1k" V 7534 850 50  0000 C CNN
-F 2 "Resistor_SMD:R_1206_3216Metric" V 7580 850 50  0001 C CNN
+F 2 "Resistor_SMD:R_1206_3216Metric_Pad1.42x1.75mm_HandSolder" V 7580 850 50  0001 C CNN
 F 3 "~" H 7650 850 50  0001 C CNN
 	1    7650 850
@@
 F 0 "R3" H 6680 954 50  0000 R CNN
 F 1 "1k" H 6680 1045 50  0000 R CNN
-F 2 "Resistor_SMD:R_1206_3216Metric" V 6680 1000 50  0001 C CNN
+F 2 "Resistor_SMD:R_1206_3216Metric_Pad1.42x1.75mm_HandSolder" V 6680 1000 50  0001 C CNN
 F 3 "~" H 6750 1000 50  0001 C CNN
 	1    6750 1000
@@
 F 0 "D1" V 4188 5533 50  0000 R CNN
 F 1 "LED" V 4097 5533 50  0000 R CNN
-F 2 "LED_SMD:LED_1206_3216Metric" H 4150 5650 50  0001 C CNN
+F 2 "LED_SMD:LED_1206_3216Metric_Pad1.42x1.75mm_HandSolder" H 4150 5650 50  0001 C CNN
 F 3 "~" H 4150 5650 50  0001 C CNN
 	1    4150 5650
@@
 F 0 "R1" H 4080 5254 50  0000 R CNN
 F 1 "1k" H 4080 5345 50  0000 R CNN
-F 2 "Resistor_SMD:R_1206_3216Metric" V 4080 5300 50  0001 C CNN
+F 2 "Resistor_SMD:R_1206_3216Metric_Pad1.42x1.75mm_HandSolder" V 4080 5300 50  0001 C CNN
 F 3 "~" H 4150 5300 50  0001 C CNN
 	1    4150 5300
@@
 F 0 "R17" V 2943 2000 50  0000 C CNN
 F 1 "0" V 3034 2000 50  0000 C CNN
-F 2 "Resistor_SMD:R_1206_3216Metric" V 3080 2000 50  0001 C CNN
+F 2 "Resistor_SMD:R_1206_3216Metric_Pad1.42x1.75mm_HandSolder" V 3080 2000 50  0001 C CNN
 F 3 "~" H 3150 2000 50  0001 C CNN
 	1    3150 2000
@@
 F 0 "C8" H 2942 5146 50  0000 L CNN
 F 1 "0.33uF" H 2942 5055 50  0000 L CNN
-F 2 "Capacitor_SMD:C_1206_3216Metric" H 2850 5100 50  0001 C CNN
+F 2 "Capacitor_SMD:C_1206_3216Metric_Pad1.42x1.75mm_HandSolder" H 2850 5100 50  0001 C CNN
 F 3 "~" H 2850 5100 50  0001 C CNN
 	1    2850 5100
@@
 F 0 "C9" H 3842 5146 50  0000 L CNN
 F 1 "0.33uF" H 3842 5055 50  0000 L CNN
-F 2 "Capacitor_SMD:C_1206_3216Metric" H 3750 5100 50  0001 C CNN
+F 2 "Capacitor_SMD:C_1206_3216Metric_Pad1.42x1.75mm_HandSolder" H 3750 5100 50  0001 C CNN
 F 3 "~" H 3750 5100 50  0001 C CNN
 	1    3750 5100
